File: MidiClockBox_v3.kicad_sch (KiCad schematic)
At the start: 89 parts, among them J1 Midi In 0, J10 Display, J11 Midi Out 3, J12 Midi Out 4, J13 Midi Out 5, J14 Sync Out 0, J15 Sync Out 1, J16 Spare, J17 Conn_01x07, J18 Conn_01x07, J19 Conn_02x05_Odd_Even, J2 ICSP, J20 Conn_02x05_Odd_Even, J3 WS2812, J4 Conn_02x07_Odd_Even, J5 Conn_02x12_Counter_Clockwise, J6 Midi Out 0, J7 Midi Out 1, J8 Midi Out 2, J9 WS2812, SW1 RotaryEncoder_Switch, SW2 TAP, SW3 Start, SW4 Stop, SW5 Preset1, SW6 Preset2, SW7 Preset3, U1 CD74HC4067SM, U2 74LS241, U3 6N138, U4 74HC595, U6 74LS08, U7 74LS08, U8 74HC595, U9 74LS241

Commit message: add title and revision to schema and pcb
Other:
- title: (none) -> Clockbox v3
Changed lines of the file:
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@@
 (kicad_sch
-	(version 20231120)
+	(version 20250114)
 	(generator "eeschema")
-	(generator_version "8.0")
+	(generator_version "9.0")
 	(paper "A3")
+	(title_block
+		(title "Clockbox v3")
+		(rev "202509001")
+	)
+	(text "Daughterboard"
+		(exclude_from_sim no)
+		(at 152.908 66.04 0)
+		(effects
+			(font
+				(size 1.27 1.27)
+			)
+		)
+	)
+	(text "Hardware midi in/ out: check\nIndependent midi out -> demultiplex: check\nsync out extra pin for START STOP: check\nboard targeted for case-use\nPotentialfreie Kontakte"
+		(exclude_from_sim no)
+		(at 349.504 261.112 0)
+		(effects
+			(font
+				(size 1.27 1.27)
+			)
+		)
+	)
+	(text "Mainboard"
+		(exclude_from_sim no)
+		(at 200.152 62.484 0)
+		(effects
+			(font
+				(size 1.27 1.27)
+			)
+		)
+	)
+	(text "Buttonboard"
+		(exclude_from_sim no)
+		(at 220.472 147.574 0)
+		(effects
+			(font
+				(size 1.27 1.27)
+			)
+		)
+	)
+	(text "SYNC START STOP sind nicht unabhängig, \naber es gibt 6 gepufferte Ausgänge mit VCC und GND\nzum Forschen"
+		(exclude_from_sim no)
+		(at 168.148 235.204 0)
+		(effects
+			(font
+				(size 1.27 1.27)
+			)
+		)
+	)
+	(text "D20 / A2"
+		(exclude_from_sim no)
+		(at 311.658 66.548 0)
+		(effects
+			(font
+				(size 1.27 1.27)
+			)
+		)
+	)
+	(text "D5"
+		(exclude_from_sim no)
+		(at 264.922 71.374 0)
+		(effects
+			(font
+				(size 1.27 1.27)
+			)
+		)
+	)
+	(text "Motherboard"
+		(exclude_from_sim no)
+		(at 220.472 124.714 0)
+		(effects
+			(font
+				(size 1.27 1.27)
+			)
+		)
+	)
+	(text "Pre-load MIDI and SYNC outputs"
+		(exclude_from_sim no)
+		(at 88.138 108.458 0)
+		(effects
+			(font
+				(size 1.27 1.27)
+			)
+		)
+	)
+	(text "D19 / A1"
+		(exclude_from_sim no)
+		(at 307.848 68.834 0)
+		(effects
+			(font
+				(size 1.27 1.27)
+			)
+		)
+	)
+	(text "D4 / A6"
+		(exclude_from_sim no)
+		(at 264.668 69.088 0)
+		(effects
+			(font
+				(size 1.27 1.27)
+			)
+		)
+	)
 	(junction
 		(at 80.01 91.44)
@@
 		)
 	)
-	(text "Daughterboard"
-		(exclude_from_sim no)
-		(at 152.908 66.04 0)
-		(effects
-			(font
-				(size 1.27 1.27)
-			)
-		)
-	)
-	(text "Hardware midi in/ out: check\nIndependent midi out -> demultiplex: check\nsync out extra pin for START STOP: check\nboard targeted for case-use\nPotentialfreie Kontakte"
-		(exclude_from_sim no)
-		(at 349.504 261.112 0)
-		(effects
-			(font
-				(size 1.27 1.27)
-			)
-		)
-	)
-	(text "Mainboard"
-		(exclude_from_sim no)
-		(at 200.152 62.484 0)
-		(effects
-			(font
-				(size 1.27 1.27)
-			)
-		)
-	)
-	(text "Buttonboard"
-		(exclude_from_sim no)
-		(at 220.472 147.574 0)
-		(effects
-			(font
-				(size 1.27 1.27)
-			)
-		)
-	)
-	(text "SYNC START STOP sind nicht unabhängig, \naber es gibt 6 gepufferte Ausgänge mit VCC und GND\nzum Forschen"
-		(exclude_from_sim no)
-		(at 168.148 235.204 0)
-		(effects
-			(font
-				(size 1.27 1.27)
-			)
-		)
-	)
-	(text "D20 / A2"
-		(exclude_from_sim no)
-		(at 311.658 66.548 0)
-		(effects
-			(font
-				(size 1.27 1.27)
-			)
-		)
-	)
-	(text "D5"
-		(exclude_from_sim no)
-		(at 264.922 71.374 0)
-		(effects
-			(font
-				(size 1.27 1.27)
-			)
-		)
-	)
-	(text "Motherboard"
-		(exclude_from_sim no)
-		(at 220.472 124.714 0)
-		(effects
-			(font
-				(size 1.27 1.27)
-			)
-		)
-	)
-	(text "Pre-load MIDI and SYNC outputs"
-		(exclude_from_sim no)
-		(at 88.138 108.458 0)
-		(effects
-			(font
-				(size 1.27 1.27)
-			)
-		)
-	)
-	(text "D19 / A1"
-		(exclude_from_sim no)
-		(at 307.848 68.834 0)
-		(effects
-			(font
-				(size 1.27 1.27)
-			)
-		)
-	)
-	(text "D4 / A6"
-		(exclude_from_sim no)
-		(at 264.668 69.088 0)
-		(effects
-			(font
-				(size 1.27 1.27)
-			)
-		)
-	)
 	(global_label "LED_DATA"
 		(shape input)
@@
 		)
 	)
+	(embedded_fonts no)
 )
